File: kicad/christmas-tree/christmas-tree.kicad_sch (KiCad schematic)
At the start: 2 parts, among them U101 Seeeduino-XIAO-ESP32C6

Commit message: test
Parts:
- removed D101: SK6812, LED_SMD:LED_SK6812_PLCC4_5.0x5.0mm_P3.2mm, symbol LED:SK6812
- added 5V1, 5V2, DIN1, DOUT1, GND1, GND2: 2.0mm, 0_lpt_misc:TestPad_2.0mm, symbol 0_lpt_misc:TestPad_2.0mm
- added C101, C102, C103, C104, C105, C106, C107, C108, C109, C110, C111, C112, C113, C114, C115, C116, C117, C118, C119, C120, C121, C122, C123: 100n X7R 50V, Resistor_SMD:R_0603_1608Metric, symbol 0_lpt_rcl:C_0603_100n_X7R_50V
- added C124: C_1206, Capacitor_SMD:C_1206_3216Metric_Pad1.33x1.80mm_HandSolder, symbol 0_lpt_rcl:C_1206
- added D101, D102, D103, D104, D105, D106, D107, D108, D109, D110, D111, D112, D113, D114, D115, D116, D117, D118, D119, D120, D121, D122, D123, D124, D125, D126, D127, D128, D129, D130, D131, D132, D133, D134, D135, D136, D137, D138, D139, D140, D141, D142, D143, D144, D145, D146: WS2812B, LED_SMD:LED_WS2812B_PLCC4_5.0x5.0mm_P3.2mm, symbol LED:WS2812B
Connections:
- net at U101.10 (D9): now also D101.4 (DIN)
- net GND: now reaches U101.13 (GND)
- net GND: now also C101.1, C102.1, C103.1, C104.1, C105.1, C106.1, C107.1, C108.1, C109.1, C110.1, C111.1, C112.1, C113.1, C114.1, C115.1, C116.1, C117.1, C118.1, C119.1, C120.1, C121.1, C122.1, C123.1, C124.2, D101.3 (VSS), D102.3 (VSS), D103.3 (VSS), D104.3 (VSS), D105.3 (VSS), D106.3 (VSS), D107.3 (VSS), D108.3 (VSS), D109.3 (VSS), D110.3 (VSS), D111.3 (VSS), D112.3 (VSS), D113.3 (VSS), D114.3 (VSS), D115.3 (VSS), D116.3 (VSS), D117.3 (VSS), D118.3 (VSS), D119.3 (VSS), D120.3 (VSS), D121.3 (VSS), D122.3 (VSS), D123.3 (VSS), D124.3 (VSS), D125.3 (VSS), D126.3 (VSS), D127.3 (VSS), D128.3 (VSS), D129.3 (VSS), D130.3 (VSS), D131.3 (VSS), D132.3 (VSS), D133.3 (VSS), D134.3 (VSS), D135.3 (VSS), D136.3 (VSS), D137.3 (VSS), D138.3 (VSS), D139.3 (VSS), D140.3 (VSS), D141.3 (VSS), D142.3 (VSS), D143.3 (VSS), D144.3 (VSS), D145.3 (VSS), D146.3 (VSS), GND1.1, GND2.1
- net 5V: now reaches U101.14 (5V)
- net 5V: now also 5V1.1, 5V2.1, C101.2, C102.2, C103.2, C104.2, C105.2, C106.2, C107.2, C108.2, C109.2, C110.2, C111.2, C112.2, C113.2, C114.2, C115.2, C116.2, C117.2, C118.2, C119.2, C120.2, C121.2, C122.2, C123.2, C124.1, D101.1 (VDD), D102.1 (VDD), D103.1 (VDD), D104.1 (VDD), D105.1 (VDD), D106.1 (VDD), D107.1 (VDD), D108.1 (VDD), D109.1 (VDD), D110.1 (VDD), D111.1 (VDD), D112.1 (VDD), D113.1 (VDD), D114.1 (VDD), D115.1 (VDD), D116.1 (VDD), D117.1 (VDD), D118.1 (VDD), D119.1 (VDD), D120.1 (VDD), D121.1 (VDD), D122.1 (VDD), D123.1 (VDD), D124.1 (VDD), D125.1 (VDD), D126.1 (VDD), D127.1 (VDD), D128.1 (VDD), D129.1 (VDD), D130.1 (VDD), D131.1 (VDD), D132.1 (VDD), D133.1 (VDD), D134.1 (VDD), D135.1 (VDD), D136.1 (VDD), D137.1 (VDD), D138.1 (VDD), D139.1 (VDD), D140.1 (VDD), D141.1 (VDD), D142.1 (VDD), D143.1 (VDD), D144.1 (VDD), D145.1 (VDD), D146.1 (VDD)
- new net: D116.2 (DOUT), D117.4 (DIN)
- new net: D115.2 (DOUT), D116.4 (DIN)
- new net: D104.2 (DOUT), D105.4 (DIN)
- new net: D103.2 (DOUT), D104.4 (DIN)
- new net: D127.2 (DOUT), D128.4 (DIN)
- new net: D126.2 (DOUT), D127.4 (DIN)
- new net: D110.2 (DOUT), D111.4 (DIN)
- new net: D109.2 (DOUT), D110.4 (DIN)
- new net: D105.2 (DOUT), D106.4 (DIN)
- new net: D102.2 (DOUT), D103.4 (DIN)
- new net: D101.2 (DOUT), D102.4 (DIN)
- new net: D136.2 (DOUT), D137.4 (DIN)
- new net: D135.2 (DOUT), D136.4 (DIN)
- new net: D132.2 (DOUT), D133.4 (DIN)
- new net: D131.2 (DOUT), D132.4 (DIN)
- new net: D140.2 (DOUT), D141.4 (DIN)
- new net: D139.2 (DOUT), D140.4 (DIN)
- new net: D145.2 (DOUT), D146.4 (DIN)
- new net: D138.2 (DOUT), D139.4 (DIN)
- new net: D137.2 (DOUT), D138.4 (DIN)
- new net: D142.2 (DOUT), D143.4 (DIN)
- new net: D141.2 (DOUT), D142.4 (DIN)
- new net: D125.2 (DOUT), D126.4 (DIN)
- new net: D117.2 (DOUT), D118.4 (DIN)
- new net: D133.2 (DOUT), D134.4 (DIN)
- new net: D114.2 (DOUT), D115.4 (DIN)
- new net: D111.2 (DOUT), D112.4 (DIN)
- new net: D119.2 (DOUT), D120.4 (DIN)
- new net: D118.2 (DOUT), D119.4 (DIN)
- new net: D129.2 (DOUT), D130.4 (DIN)
- new net: D128.2 (DOUT), D129.4 (DIN)
- new net: D121.2 (DOUT), D122.4 (DIN)
- new net: D120.2 (DOUT), D121.4 (DIN)
- new net: D130.2 (DOUT), D131.4 (DIN)
- new net: D122.2 (DOUT), DOUT1.1
- new net: D144.2 (DOUT), D145.4 (DIN)
- new net: D134.2 (DOUT), D135.4 (DIN)
- new net: D124.2 (DOUT), D125.4 (DIN)
- new net: D123.2 (DOUT), D124.4 (DIN)
- new net: D108.2 (DOUT), D109.4 (DIN)
- new net: D107.2 (DOUT), D108.4 (DIN)
- new net: D143.2 (DOUT), D144.4 (DIN)
- new net: D123.4 (DIN), DIN1.1
- new net: D106.2 (DOUT), D107.4 (DIN)
- new net: D113.2 (DOUT), D114.4 (DIN)
- new net: D112.2 (DOUT), D113.4 (DIN)
Other:
- moved on the sheet: U101
